Commit message: Adding model urdf visualization

File: model.urdf (robot description, URDF)
Before this commit: robot my_maze, 99 links, 98 joints
Links:
- link wall1: geometry collision box size=0.05 0.55 0.3; visual box size=0.05 0.55 0.3
- link wall10: geometry collision box size=0.05 0.55 0.3
- link wall11: geometry collision box size=0.05 0.55 0.3
- link wall12: geometry collision box size=0.05 0.55 0.3
- link wall13: geometry collision box size=0.05 0.55 0.3
- link wall14: geometry collision box size=0.05 0.55 0.3
- link wall15: geometry collision box size=0.05 0.55 0.3
- link wall16: geometry collision box size=0.05 0.55 0.3
- link wall17: geometry collision box size=0.05 0.55 0.3
- link wall18: geometry collision box size=0.05 0.55 0.3
- link wall19: geometry collision box size=0.05 0.55 0.3
- link wall2: geometry collision box size=0.05 0.55 0.3
- link wall20: geometry collision box size=0.05 0.55 0.3
- link wall21: geometry collision box size=0.05 0.55 0.3
- link wall22: geometry collision box size=0.05 0.55 0.3
- link wall23: geometry collision box size=0.05 0.55 0.3
- link wall24: geometry collision box size=0.05 0.55 0.3
- link wall25: geometry collision box size=0.05 0.55 0.3
- link wall26: geometry collision box size=0.05 0.55 0.3
- link wall27: geometry collision box size=0.05 0.55 0.3
- link wall28: geometry collision box size=0.05 0.55 0.3
- link wall29: geometry collision box size=0.05 0.55 0.3
- link wall3: geometry collision box size=0.05 0.55 0.3
- link wall30: geometry collision box size=0.05 0.55 0.3
- link wall31: geometry collision box size=0.05 0.55 0.3
- link wall32: geometry collision box size=0.05 0.55 0.3
- link wall33: geometry collision box size=0.05 0.55 0.3
- link wall34: geometry collision box size=0.05 0.55 0.3
- link wall35: geometry collision box size=0.05 0.55 0.3
- link wall36: geometry collision box size=0.05 0.55 0.3
- link wall37: geometry collision box size=0.05 0.55 0.3
- link wall38: geometry collision box size=0.05 0.55 0.3
- link wall39: geometry collision box size=0.05 0.55 0.3
- link wall4: geometry collision box size=0.05 0.55 0.3
- link wall40: geometry collision box size=0.05 0.55 0.3
- link wall41: geometry collision box size=0.05 0.55 0.3
- link wall42: geometry collision box size=0.05 0.55 0.3
- link wall43: geometry collision box size=0.05 0.55 0.3
- link wall44: geometry collision box size=0.05 0.55 0.3
- link wall45: geometry collision box size=0.05 0.55 0.3
- link wall46: geometry collision box size=0.05 0.55 0.3
- link wall47: geometry collision box size=0.05 0.55 0.3
- link wall48: geometry collision box size=0.05 0.55 0.3
- link wall49: geometry collision box size=0.05 0.55 0.3
- link wall5: geometry collision box size=0.05 0.55 0.3
- link wall50: geometry collision box size=0.05 0.55 0.3
- link wall51: geometry collision box size=0.05 0.55 0.3
- link wall52: geometry collision box size=0.05 0.55 0.3
- link wall53: geometry collision box size=0.05 0.55 0.3
- link wall54: geometry collision box size=0.05 0.55 0.3
- link wall55: geometry collision box size=0.05 0.55 0.3
- link wall56: geometry collision box size=0.05 0.55 0.3
- link wall57: geometry collision box size=0.05 0.55 0.3
- link wall58: geometry collision box size=0.05 0.55 0.3
- link wall59: geometry collision box size=0.05 0.55 0.3
- link wall6: geometry collision box size=0.05 0.55 0.3
- link wall60: geometry collision box size=0.05 0.55 0.3
- link wall61: geometry collision box size=0.05 0.55 0.3
- link wall62: geometry collision box size=0.05 0.55 0.3
- link wall63: geometry collision box size=0.05 0.55 0.3
- link wall64: geometry collision box size=0.05 0.55 0.3
- link wall65: geometry collision box size=0.05 0.55 0.3
- link wall66: geometry collision box size=0.05 0.55 0.3
- link wall67: geometry collision box size=0.05 0.55 0.3
- link wall68: geometry collision box size=0.05 0.55 0.3
- link wall69: geometry collision box size=0.05 0.55 0.3
- link wall7: geometry collision box size=0.05 0.55 0.3
- link wall70: geometry collision box size=0.05 0.55 0.3
- link wall71: geometry collision box size=0.05 0.55 0.3
- link wall72: geometry collision box size=0.05 0.55 0.3
- link wall73: geometry collision box size=0.05 0.55 0.3
- link wall74: geometry collision box size=0.05 0.55 0.3
- link wall75: geometry collision box size=0.05 0.55 0.3
- link wall76: geometry collision box size=0.05 0.55 0.3
- link wall77: geometry collision box size=0.05 0.55 0.3
- link wall78: geometry collision box size=0.05 0.55 0.3
- link wall79: geometry collision box size=0.05 0.55 0.3
- link wall8: geometry collision box size=0.05 0.55 0.3
- link wall80: geometry collision box size=0.05 0.55 0.3
- link wall81: geometry collision box size=0.05 0.55 0.3
- link wall82: geometry collision box size=0.05 0.55 0.3
- link wall83: geometry collision box size=0.05 0.55 0.3
- link wall84: geometry collision box size=0.05 0.55 0.3
- link wall85: geometry collision box size=0.05 0.55 0.3
- link wall86: geometry collision box size=0.05 0.55 0.3
- link wall87: geometry collision box size=0.05 0.55 0.3
- link wall88: geometry collision box size=0.05 0.55 0.3
- link wall89: geometry collision box size=0.05 0.55 0.3
- link wall9: geometry collision box size=0.05 0.55 0.3
- link wall90: geometry collision box size=0.05 0.55 0.3
- link wall91: geometry collision box size=0.05 0.55 0.3
- link wall92: geometry collision box size=0.05 0.55 0.3
- link wall93: geometry collision box size=0.05 0.55 0.3
- link wall94: geometry collision box size=0.05 0.55 0.3
- link wall95: geometry collision box size=0.05 0.55 0.3
- link wall96: geometry collision box size=0.05 0.55 0.3
- link wall97: geometry collision box size=0.05 0.55 0.3
- link wall98: geometry collision box size=0.05 0.55 0.3
