Commit message: added correct urdf

File: dev_test_urdf/Nitya/Final/assets/room.urdf (robot description, URDF)
Before this commit: robot room, 9 links, 8 joints
Links:
- removed link wall4
- added link wall4a; collision box size=5 0.2 0.7; visual box size=5 0.2 0.7
- added link wall4b; collision box size=5 0.2 0.7; visual box size=5 0.2 0.7
- added link wall4c; collision box size=1.5 0.2 0.6; visual box size=1.5 0.2 0.6
- added link wall4d; collision box size=1.5 0.2 0.6; visual box size=1.5 0.2 0.6
- link ground1: geometry collision box size=2.5 2.5 0.1; visual box size=2.5 2.5 0.1
- link ground2: geometry collision box size=2.5 2.5 0.1; visual box size=2.5 2.5 0.1
- link ground3: geometry collision box size=2.5 2.5 0.1; visual box size=2.5 2.5 0.1
- link wall1: geometry collision box size=5 0.2 2; visual box size=5 0.2 2
- link wall2: geometry collision box size=0.2 5 2; visual box size=0.2 5 2
- link wall3: geometry collision box size=0.2 5 2; visual box size=0.2 5 2
- link wall5: geometry collision box size=3.75 0.2 2; visual box size=3.75 0.2 2
Joints:
- removed joint wall4
- added joint wall4a: type fixed, parent odom, child wall4a
- added joint wall4b: type fixed, parent odom, child wall4b
- added joint wall4c: type fixed, parent odom, child wall4c
- added joint wall4d: type fixed, parent odom, child wall4d

Commit message: changed window height

File: dev_test_urdf/Nitya/Final/assets/room.urdf (robot description, URDF)
Before this commit: robot room, 12 links, 11 joints
Links:
- link wall4a: geometry collision box size=5 0.2 0.5; visual box size=5 0.2 0.5
- link wall4b: geometry collision box size=5 0.2 0.5; visual box size=5 0.2 0.5
- link wall4c: geometry collision box size=1.5 0.2 1; visual box size=1.5 0.2 1
- link wall4d: geometry collision box size=1.5 0.2 1; visual box size=1.5 0.2 1

Commit message: room change

File: dev_test_urdf/Nitya/Final/assets/room.urdf (robot description, URDF)
Before this commit: robot room, 12 links, 11 joints
Links:
- link wall5: geometry collision box size=3 0.2 2; visual box size=3 0.2 2
